File: kicad/choc/sha-choc.kicad_sch (KiCad schematic)
At the start: 111 parts, among them SW1 SW_Push, SW10 SW_Push, SW11 SW_Push, SW12 SW_Push, SW13 SW_Push, SW14 SW_Push, SW15 SW_Push, SW16 SW_Push, SW17 SW_Push, SW18 SW_Push, SW19 SW_Push, SW2 SW_Push, SW20 SW_Push, SW21 SW_Push, SW22 SW_Push, SW23 SW_Push, SW24 SW_Push, SW25 SW_Push, SW26 SW_Push, SW27 SW_Push, SW28 SW_Push, SW29 SW_Push, SW3 SW_Push, SW30 SW_Push, SW31 SW_Push, SW32 SW_Push, SW33 SW_Push, SW34 SW_Push, SW35 SW_Push, SW36 SW_Push, SW37 SW_Push, SW38 SW_Push, SW39 SW_Push, SW4 SW_Push, SW40 SW_Push, SW41 SW_Push, SW42 SW_Push, SW43 SW_Push, SW44 SW_Push, SW45 SW_Push, SW46 SW_Push, SW47 SW_Push, SW48 SW_Push, SW49 SW_Push, SW5 SW_Push, SW50 SW_Push, SW6 SW_Push, SW7 SW_Push, SW8 SW_Push, SW9 SW_Push, U1 RP2040-Zero

Commit message: Create Choc switch design, update logos
Parts:
- SW1, SW10, SW11, SW12, SW13, SW14, SW15, SW16, SW17, SW18, SW19, SW2, SW20, SW21, SW22, SW23, SW24, SW25, SW26, SW27, SW28, SW29, SW3, SW30, SW31, SW32, SW33, SW34, SW35, SW36, SW37, SW38, SW39, SW4, SW40, SW41, SW42, SW43, SW44, SW45, SW46, SW47, SW48, SW49, SW5, SW50, SW6, SW7, SW8, SW9: footprint sha-footprints:SW_MX_Reverse_Cutout -> sha-footprints:SW_Choc_Reverse_Cutout
Other:
- title: Sha MX -> Sha Choc
Changed lines of the file:
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@@
 	(paper "A4")
 	(title_block
-		(title "Sha MX")
+		(title "Sha Choc")
 		(date "2024-10-09")
 		(rev "1.1")
@@
 			)
 		)
-		(property "Footprint" "sha-footprints:SW_MX_Reverse_Cutout"
+		(property "Footprint" "sha-footprints:SW_Choc_Reverse_Cutout"
 			(at 91.44 64.77 0)
 			(effects
@@
 			)
 		)
-		(property "Footprint" "sha-footprints:SW_MX_Reverse_Cutout"
+		(property "Footprint" "sha-footprints:SW_Choc_Reverse_Cutout"
 			(at 210.82 50.8 0)
 			(effects
@@
 			)
 		)
-		(property "Footprint" "sha-footprints:SW_MX_Reverse_Cutout"
+		(property "Footprint" "sha-footprints:SW_Choc_Reverse_Cutout"
 			(at 157.48 78.74 0)
 			(effects
@@
 			)
 		)
-		(property "Footprint" "sha-footprints:SW_MX_Reverse_Cutout"
+		(property "Footprint" "sha-footprints:SW_Choc_Reverse_Cutout"
 			(at 210.82 78.74 0)
 			(effects
@@
 			)
 		)
-		(property "Footprint" "sha-footprints:SW_MX_Reverse_Cutout"
+		(property "Footprint" "sha-footprints:SW_Choc_Reverse_Cutout"
 			(at 264.16 78.74 0)
 			(effects
@@
 			)
 		)
-		(property "Footprint" "sha-footprints:SW_MX_Reverse_Cutout"
+		(property "Footprint" "sha-footprints:SW_Choc_Reverse_Cutout"
 			(at 38.1 36.83 0)
 			(effects
@@
 			)
 		)
-		(property "Footprint" "sha-footprints:SW_MX_Reverse_Cutout"
+		(property "Footprint" "sha-footprints:SW_Choc_Reverse_Cutout"
 			(at 55.88 50.8 0)
 			(effects
@@
 			)
 		)
-		(property "Footprint" "sha-footprints:SW_MX_Reverse_Cutout"
+		(property "Footprint" "sha-footprints:SW_Choc_Reverse_Cutout"
 			(at 38.1 64.77 0)
 			(effects
@@
 			)
 		)
-		(property "Footprint" "sha-footprints:SW_MX_Reverse_Cutout"
+		(property "Footprint" "sha-footprints:SW_Choc_Reverse_Cutout"
 			(at 109.22 78.74 0)
 			(effects
@@
 			)
 		)
-		(property "Footprint" "sha-footprints:SW_MX_Reverse_Cutout"
+		(property "Footprint" "sha-footprints:SW_Choc_Reverse_Cutout"
 			(at 91.44 78.74 0)
 			(effects
@@
 			)
 		)
-		(property "Footprint" "sha-footprints:SW_MX_Reverse_Cutout"
+		(property "Footprint" "sha-footprints:SW_Choc_Reverse_Cutout"
 			(at 264.16 50.8 0)
 			(effects
@@
 			)
 		)
-		(property "Footprint" "sha-footprints:SW_MX_Reverse_Cutout"
+		(property "Footprint" "sha-footprints:SW_Choc_Reverse_Cutout"
 			(at 20.32 36.83 0)
 			(effects
@@
 			)
 		)
-		(property "Footprint" "sha-footprints:SW_MX_Reverse_Cutout"
+		(property "Footprint" "sha-footprints:SW_Choc_Reverse_Cutout"
 			(at 175.26 78.74 0)
 			(effects
@@
 			)
 		)
-		(property "Footprint" "sha-footprints:SW_MX_Reverse_Cutout"
+		(property "Footprint" "sha-footprints:SW_Choc_Reverse_Cutout"
 			(at 193.04 78.74 0)
 			(effects
@@
 			)
 		)
-		(property "Footprint" "sha-footprints:SW_MX_Reverse_Cutout"
+		(property "Footprint" "sha-footprints:SW_Choc_Reverse_Cutout"
 			(at 175.26 36.83 0)
 			(effects
@@
 			)
 		)
-		(property "Footprint" "sha-footprints:SW_MX_Reverse_Cutout"
+		(property "Footprint" "sha-footprints:SW_Choc_Reverse_Cutout"
 			(at 246.38 50.8 0)
 			(effects
@@
 			)
 		)
-		(property "Footprint" "sha-footprints:SW_MX_Reverse_Cutout"
+		(property "Footprint" "sha-footprints:SW_Choc_Reverse_Cutout"
 			(at 193.04 36.83 0)
 			(effects
@@
 			)
 		)
-		(property "Footprint" "sha-footprints:SW_MX_Reverse_Cutout"
+		(property "Footprint" "sha-footprints:SW_Choc_Reverse_Cutout"
 			(at 264.16 36.83 0)
 			(effects
@@
 			)
 		)
-		(property "Footprint" "sha-footprints:SW_MX_Reverse_Cutout"
+		(property "Footprint" "sha-footprints:SW_Choc_Reverse_Cutout"
 			(at 55.88 64.77 0)
 			(effects
@@
 			)
 		)
-		(property "Footprint" "sha-footprints:SW_MX_Reverse_Cutout"
+		(property "Footprint" "sha-footprints:SW_Choc_Reverse_Cutout"
 			(at 20.32 50.8 0)
 			(effects
@@
 			)
 		)
-		(property "Footprint" "sha-footprints:SW_MX_Reverse_Cutout"
+		(property "Footprint" "sha-footprints:SW_Choc_Reverse_Cutout"
 			(at 73.66 50.8 0)
 			(effects
@@
 			)
 		)
-		(property "Footprint" "sha-footprints:SW_MX_Reverse_Cutout"
+		(property "Footprint" "sha-footprints:SW_Choc_Reverse_Cutout"
 			(at 246.38 64.77 0)
 			(effects
@@
 			)
 		)
-		(property "Footprint" "sha-footprints:SW_MX_Reverse_Cutout"
+		(property "Footprint" "sha-footprints:SW_Choc_Reverse_Cutout"
 			(at 228.6 36.83 0)
 			(effects
@@
 			)
 		)
-		(property "Footprint" "sha-footprints:SW_MX_Reverse_Cutout"
+		(property "Footprint" "sha-footprints:SW_Choc_Reverse_Cutout"
 			(at 73.66 64.77 0)
 			(effects
@@
 			)
 		)
-		(property "Footprint" "sha-footprints:SW_MX_Reverse_Cutout"
+		(property "Footprint" "sha-footprints:SW_Choc_Reverse_Cutout"
 			(at 55.88 36.83 0)
 			(effects
@@
 			)
 		)
-		(property "Footprint" "sha-footprints:SW_MX_Reverse_Cutout"
+		(property "Footprint" "sha-footprints:SW_Choc_Reverse_Cutout"
 			(at 73.66 78.74 0)
 			(effects
@@
 			)
 		)
-		(property "Footprint" "sha-footprints:SW_MX_Reverse_Cutout"
+		(property "Footprint" "sha-footprints:SW_Choc_Reverse_Cutout"
 			(at 109.22 64.77 0)
 			(effects
@@
 			)
 		)
-		(property "Footprint" "sha-footprints:SW_MX_Reverse_Cutout"
+		(property "Footprint" "sha-footprints:SW_Choc_Reverse_Cutout"
 			(at 38.1 50.8 0)
 			(effects
@@
 			)
 		)
-		(property "Footprint" "sha-footprints:SW_MX_Reverse_Cutout"
+		(property "Footprint" "sha-footprints:SW_Choc_Reverse_Cutout"
 			(at 210.82 64.77 0)
 			(effects
@@
 			)
 		)
-		(property "Footprint" "sha-footprints:SW_MX_Reverse_Cutout"
+		(property "Footprint" "sha-footprints:SW_Choc_Reverse_Cutout"
 			(at 228.6 50.8 0)
 			(effects
@@
 			)
 		)
-		(property "Footprint" "sha-footprints:SW_MX_Reverse_Cutout"
+		(property "Footprint" "sha-footprints:SW_Choc_Reverse_Cutout"
 			(at 264.16 64.77 0)
 			(effects
@@
 			)
 		)
-		(property "Footprint" "sha-footprints:SW_MX_Reverse_Cutout"
+		(property "Footprint" "sha-footprints:SW_Choc_Reverse_Cutout"
 			(at 246.38 36.83 0)
 			(effects
@@
 			)
 		)
-		(property "Footprint" "sha-footprints:SW_MX_Reverse_Cutout"
+		(property "Footprint" "sha-footprints:SW_Choc_Reverse_Cutout"
 			(at 91.44 36.83 0)
 			(effects
@@
 			)
 		)
-		(property "Footprint" "sha-footprints:SW_MX_Reverse_Cutout"
+		(property "Footprint" "sha-footprints:SW_Choc_Reverse_Cutout"
 			(at 193.04 64.77 0)
 			(effects
@@
 			)
 		)
-		(property "Footprint" "sha-footprints:SW_MX_Reverse_Cutout"
+		(property "Footprint" "sha-footprints:SW_Choc_Reverse_Cutout"
 			(at 38.1 78.74 0)
 			(effects
@@
 			)
 		)
-		(property "Footprint" "sha-footprints:SW_MX_Reverse_Cutout"
+		(property "Footprint" "sha-footprints:SW_Choc_Reverse_Cutout"
 			(at 193.04 50.8 0)
 			(effects
@@
 			)
 		)
-		(property "Footprint" "sha-footprints:SW_MX_Reverse_Cutout"
+		(property "Footprint" "sha-footprints:SW_Choc_Reverse_Cutout"
 			(at 55.88 78.74 0)
 			(effects
@@
 			)
 		)
-		(property "Footprint" "sha-footprints:SW_MX_Reverse_Cutout"
+		(property "Footprint" "sha-footprints:SW_Choc_Reverse_Cutout"
 			(at 20.32 64.77 0)
 			(effects
@@
 			)
 		)
-		(property "Footprint" "sha-footprints:SW_MX_Reverse_Cutout"
+		(property "Footprint" "sha-footprints:SW_Choc_Reverse_Cutout"
 			(at 109.22 36.83 0)
 			(effects
@@
 			)
 		)
-		(property "Footprint" "sha-footprints:SW_MX_Reverse_Cutout"
+		(property "Footprint" "sha-footprints:SW_Choc_Reverse_Cutout"
 			(at 20.32 78.74 0)
 			(effects
@@
 			)
 		)
-		(property "Footprint" "sha-footprints:SW_MX_Reverse_Cutout"
+		(property "Footprint" "sha-footprints:SW_Choc_Reverse_Cutout"
 			(at 175.26 50.8 0)
 			(effects
@@
 			)
 		)
-		(property "Footprint" "sha-footprints:SW_MX_Reverse_Cutout"
+		(property "Footprint" "sha-footprints:SW_Choc_Reverse_Cutout"
 			(at 73.66 36.83 0)
 			(effects
@@
 			)
 		)
-		(property "Footprint" "sha-footprints:SW_MX_Reverse_Cutout"
+		(property "Footprint" "sha-footprints:SW_Choc_Reverse_Cutout"
 			(at 127 78.74 0)
 			(effects
@@
 			)
 		)
-		(property "Footprint" "sha-footprints:SW_MX_Reverse_Cutout"
+		(property "Footprint" "sha-footprints:SW_Choc_Reverse_Cutout"
 			(at 228.6 64.77 0)
 			(effects
@@
 			)
 		)
-		(property "Footprint" "sha-footprints:SW_MX_Reverse_Cutout"
+		(property "Footprint" "sha-footprints:SW_Choc_Reverse_Cutout"
 			(at 228.6 78.74 0)
 			(effects
@@
 			)
 		)
-		(property "Footprint" "sha-footprints:SW_MX_Reverse_Cutout"
+		(property "Footprint" "sha-footprints:SW_Choc_Reverse_Cutout"
 			(at 210.82 36.83 0)
 			(effects
@@
 			)
 		)
-		(property "Footprint" "sha-footprints:SW_MX_Reverse_Cutout"
+		(property "Footprint" "sha-footprints:SW_Choc_Reverse_Cutout"
 			(at 246.38 78.74 0)
 			(effects
@@
 			)
 		)
-		(property "Footprint" "sha-footprints:SW_MX_Reverse_Cutout"
+		(property "Footprint" "sha-footprints:SW_Choc_Reverse_Cutout"
 			(at 91.44 50.8 0)
 			(effects
@@
 			)
 		)
-		(property "Footprint" "sha-footprints:SW_MX_Reverse_Cutout"
+		(property "Footprint" "sha-footprints:SW_Choc_Reverse_Cutout"
 			(at 175.26 64.77 0)
 			(effects
@@
 			)
 		)
-		(property "Footprint" "sha-footprints:SW_MX_Reverse_Cutout"
+		(property "Footprint" "sha-footprints:SW_Choc_Reverse_Cutout"
 			(at 109.22 50.8 0)
 			(effects
